File: pcb/load_cell_amp_diy.brd (EAGLE design)
At the start: 49.6 x 39.6 mm, 11 parts, among them IC1 INA122P, J1 LOAD_CELL, J2 G29

Commit message: updated diy board to help etching and soldering
Changed lines of the file:
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@@
 <layers>
 <layer number="1" name="Top" color="4" fill="1" visible="no" active="yes"/>
-<layer number="16" name="Bottom" color="60" fill="1" visible="yes" active="yes"/>
-<layer number="17" name="Pads" color="60" fill="1" visible="yes" active="yes"/>
+<layer number="16" name="Bottom" color="2" fill="1" visible="yes" active="yes"/>
+<layer number="17" name="Pads" color="52" fill="1" visible="yes" active="yes"/>
 <layer number="18" name="Vias" color="2" fill="1" visible="no" active="yes"/>
 <layer number="19" name="Unrouted" color="6" fill="1" visible="no" active="yes"/>
@@
 <layer number="114" name="Badge_Outline" color="7" fill="1" visible="no" active="no"/>
 <layer number="115" name="ReferenceISLANDS" color="7" fill="1" visible="no" active="no"/>
-<layer number="116" name="centerDrill" color="0" fill="1" visible="yes" active="yes"/>
+<layer number="116" name="centerDrill" color="57" fill="1" visible="no" active="yes"/>
 <layer number="117" name="PM_Ref" color="7" fill="1" visible="no" active="no"/>
 <layer number="118" name="Rect_Pads" color="7" fill="1" visible="no" active="no"/>
@@
 <text x="54.483" y="36.83" size="0.8128" layer="25">BRAKE</text>
 <text x="54.356" y="34.29" size="0.8128" layer="25">CLUTCH</text>
-<circle x="44.704" y="34.163" radius="0.275" width="0.55" layer="116"/>
-<circle x="44.704" y="30.353" radius="0.275" width="0.55" layer="116"/>
-<circle x="45.339" y="45.974" radius="0.275" width="0.55" layer="116"/>
-<circle x="45.339" y="43.434" radius="0.275" width="0.55" layer="116"/>
-<circle x="45.339" y="40.894" radius="0.275" width="0.55" layer="116"/>
-<circle x="45.339" y="38.354" radius="0.275" width="0.55" layer="116"/>
-<circle x="52.959" y="38.354" radius="0.275" width="0.55" layer="116"/>
-<circle x="52.959" y="40.894" radius="0.275" width="0.55" layer="116"/>
-<circle x="52.959" y="43.434" radius="0.275" width="0.55" layer="116"/>
-<circle x="52.959" y="45.974" radius="0.275" width="0.55" layer="116"/>
-<circle x="29.591" y="38.227" radius="0.275" width="0.55" layer="116"/>
-<circle x="29.591" y="40.767" radius="0.275" width="0.55" layer="116"/>
-<circle x="29.591" y="43.307" radius="0.275" width="0.55" layer="116"/>
-<circle x="29.591" y="45.847" radius="0.275" width="0.55" layer="116"/>
-<circle x="66.421" y="43.561" radius="0.275" width="0.55" layer="116"/>
-<circle x="66.421" y="41.021" radius="0.275" width="0.55" layer="116"/>
-<circle x="66.421" y="38.481" radius="0.275" width="0.55" layer="116"/>
-<circle x="66.421" y="35.941" radius="0.275" width="0.55" layer="116"/>
-<circle x="39.37" y="33.02" radius="0.275" width="0.55" layer="116"/>
-<circle x="39.37" y="43.18" radius="0.275" width="0.55" layer="116"/>
-<circle x="35.654" y="51.059" radius="0.275" width="0.55" layer="116"/>
-<circle x="35.654" y="40.899" radius="0.275" width="0.55" layer="116"/>
-<circle x="58.039" y="38.354" radius="0.275" width="0.55" layer="116"/>
-<circle x="58.039" y="48.514" radius="0.275" width="0.55" layer="116"/>
-<circle x="61.468" y="28.194" radius="0.275" width="0.55" layer="116"/>
-<circle x="61.468" y="38.354" radius="0.275" width="0.55" layer="116"/>
-<circle x="38.349" y="56.515" radius="0.275" width="0.55" layer="116"/>
-<circle x="33.269" y="56.515" radius="0.275" width="0.55" layer="116"/>
-<circle x="35.809" y="56.515" radius="0.275" width="0.55" layer="116"/>
-<circle x="52.197" y="52.578" radius="0.275" width="0.55" layer="116"/>
-<circle x="47.117" y="52.578" radius="0.275" width="0.55" layer="116"/>
-<circle x="49.657" y="52.578" radius="0.275" width="0.55" layer="116"/>
-<circle x="55.626" y="32.512" radius="0.275" width="0.55" layer="116"/>
-<circle x="50.546" y="32.512" radius="0.275" width="0.55" layer="116"/>
-<circle x="53.086" y="32.512" radius="0.275" width="0.55" layer="116"/>
+<circle x="44.704" y="34.163" radius="0.05" width="0.55" layer="116"/>
+<circle x="44.704" y="30.353" radius="0.05" width="0.55" layer="116"/>
+<circle x="45.339" y="45.974" radius="0.05" width="0.55" layer="116"/>
+<circle x="45.339" y="43.434" radius="0.05" width="0.55" layer="116"/>
+<circle x="45.339" y="40.894" radius="0.05" width="0.55" layer="116"/>
+<circle x="45.339" y="38.354" radius="0.05" width="0.55" layer="116"/>
+<circle x="52.959" y="38.354" radius="0.05" width="0.55" layer="116"/>
+<circle x="52.959" y="40.894" radius="0.05" width="0.55" layer="116"/>
+<circle x="52.959" y="43.434" radius="0.05" width="0.55" layer="116"/>
+<circle x="52.959" y="45.974" radius="0.05" width="0.55" layer="116"/>
+<circle x="29.591" y="38.227" radius="0.05" width="0.55" layer="116"/>
+<circle x="29.591" y="40.767" radius="0.05" width="0.55" layer="116"/>
+<circle x="29.591" y="43.307" radius="0.05" width="0.55" layer="116"/>
+<circle x="29.591" y="45.847" radius="0.05" width="0.55" layer="116"/>
+<circle x="66.421" y="43.561" radius="0.05" width="0.55" layer="116"/>
+<circle x="66.421" y="41.021" radius="0.05" width="0.55" layer="116"/>
+<circle x="66.421" y="38.481" radius="0.05" width="0.55" layer="116"/>
+<circle x="66.421" y="35.941" radius="0.05" width="0.55" layer="116"/>
+<circle x="39.37" y="33.02" radius="0.05" width="0.55" layer="116"/>
+<circle x="39.37" y="43.18" radius="0.05" width="0.55" layer="116"/>
+<circle x="35.654" y="51.059" radius="0.05" width="0.55" layer="116"/>
+<circle x="35.654" y="40.899" radius="0.05" width="0.55" layer="116"/>
+<circle x="58.039" y="38.354" radius="0.05" width="0.55" layer="116"/>
+<circle x="58.039" y="48.514" radius="0.05" width="0.55" layer="116"/>
+<circle x="61.468" y="28.194" radius="0.05" width="0.55" layer="116"/>
+<circle x="61.468" y="38.354" radius="0.05" width="0.55" layer="116"/>
+<circle x="38.349" y="56.515" radius="0.05" width="0.55" layer="116"/>
+<circle x="33.269" y="56.515" radius="0.05" width="0.55" layer="116"/>
+<circle x="35.809" y="56.515" radius="0.05" width="0.55" layer="116"/>
+<circle x="52.197" y="52.578" radius="0.05" width="0.55" layer="116"/>
+<circle x="47.117" y="52.578" radius="0.05" width="0.55" layer="116"/>
+<circle x="49.657" y="52.578" radius="0.05" width="0.55" layer="116"/>
+<circle x="55.626" y="32.512" radius="0.05" width="0.55" layer="116"/>
+<circle x="50.546" y="32.512" radius="0.05" width="0.55" layer="116"/>
+<circle x="53.086" y="32.512" radius="0.05" width="0.55" layer="116"/>
 </plain>
 <attributes>
@@
 <contactref element="R3" pad="2"/>
 <contactref element="R_REF" pad="E"/>
-<wire x1="50.546" y1="42.418" x2="51.562" y2="43.434" width="1.27" layer="16"/>
-<wire x1="51.562" y1="43.434" x2="52.959" y2="43.434" width="1.27" layer="16"/>
+<wire x1="49.149" y1="41.529" x2="51.054" y2="43.434" width="1.27" layer="16"/>
+<wire x1="51.054" y1="43.434" x2="52.959" y2="43.434" width="1.27" layer="16"/>
 <contactref element="J1" pad="4"/>
 <wire x1="29.591" y1="45.847" x2="29.5736" y2="45.8644" width="1.27" layer="16"/>
@@
 <wire x1="52.959" y1="43.434" x2="63.119" y2="43.434" width="1.27" layer="16"/>
 <wire x1="66.294" y1="43.434" x2="66.421" y2="43.561" width="1.27" layer="16"/>
-<wire x1="44.704" y1="34.163" x2="45.72" y2="34.163" width="1.27" layer="16"/>
-<wire x1="45.72" y1="34.163" x2="50.546" y2="38.989" width="1.27" layer="16"/>
-<wire x1="50.546" y1="38.989" x2="50.546" y2="42.418" width="1.27" layer="16"/>
-<wire x1="50.546" y1="38.989" x2="50.546" y2="32.512" width="1.27" layer="16"/>
+<wire x1="44.704" y1="34.163" x2="46.482" y2="34.163" width="1.27" layer="16"/>
+<wire x1="46.482" y1="34.163" x2="49.149" y2="36.83" width="1.27" layer="16"/>
+<wire x1="49.149" y1="35.814" x2="49.149" y2="41.529" width="1.27" layer="16"/>
+<wire x1="49.149" y1="36.83" x2="49.149" y2="33.909" width="1.27" layer="16"/>
+<wire x1="49.149" y1="33.909" x2="50.546" y2="32.512" width="1.27" layer="16"/>
 <wire x1="58.039" y1="48.514" x2="63.119" y2="43.434" width="1.27" layer="16"/>
 <wire x1="63.119" y1="43.434" x2="66.294" y2="43.434" width="1.27" layer="16"/>
+<wire x1="49.149" y1="35.814" x2="50.546" y2="32.512" width="0" layer="19" extent="16-16"/>
 </signal>
 <signal name="N$6">
